File: Hardware/MidiMonger_controls.kicad_pcb (KiCad board)
At the start: 2 copper layers, 40 x 110 mm, 31 parts, among them J10 Gate8_Out, J11 CV1_Out, J12 CV2_Out, J13 CV3_Out, J14 CV4_Out, J15 USB_B_Wurth, J16 MIDI_DIN, J2 Gate3_Out, J20 Conn_01x08_Female, J21 Conn_01x08_Female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

Commit message: First completed draft of PCB electronic layout
Connections:
- J20 pad 1: CV1_LED_OUT -> CV1_OUT
- J20 pad 2: CV1_OUT -> CV2_OUT
- J20 pad 3: CV2_LED_OUT -> CV3_OUT
- J20 pad 4: CV2_OUT -> CV4_OUT
- J20 pad 5: CV3_OUT -> CV1_LED_OUT
- J20 pad 6: CV3_LED_OUT -> CV2_LED_OUT
- J20 pad 7: CV4_OUT -> CV3_LED_OUT
- J22 pad 1: GND -> RESET_SWITCH
- J22 pad 3: GATE7_LED_OUT -> GND
- J22 pad 7: USB_DM -> USB_DP
- J22 pad 8: USB_DP -> USB_DM
- J23 pad 1: GND -> GATE7_LED_OUT
- J23 pad 6: RESET_SWITCH -> GND
Routing:
- net GATE7_LED_OUT: track 16.1 -> 36.5 mm
- net GND: track 0.00 -> 13.5 mm
- net CV1_LED_OUT: track 7.49 -> 17.6 mm
- net CV4_OUT: track 27.9 -> 35.5 mm
- net CV3_OUT: track 20.0 -> 27.5 mm
- net CV2_OUT: track 13.1 -> 16.9 mm
- net CV2_LED_OUT: track 4.28 -> 7.19 mm
- net RESET_SWITCH: track 25.2 -> 22.5 mm
- net CV3_LED_OUT: track 8.71 -> 6.20 mm
- net CV1_OUT: track 12.1 -> 10.6 mm
- net USB_DM: track 9.64 -> 8.59 mm
