File: Hardware/MidiMonger.kicad_pcb (KiCad board)
At the start: 2 copper layers, 40 x 110 mm, 56 parts, among them J1 SWD_Header, J2 Conn_01x08_Male, J3 Conn_01x08_Male, J4 Conn_01x08_Male, J5 Conn_01x08_Male, J9 Eurorack_10_pin_power, U1 STM32F446RETx, U2 6N137, U3 TL074, U4 LM1117-5.0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

Commit message: First completed draft of PCB electronic layout
Parts:
- moved C8 55.8 mm to (101.3, 84.3), turned to 90 degrees
- moved R21 48.3 mm to (128.6, 81.8), turned to 180 degrees
- moved R20 26.0 mm to (130.2, 95.0), turned to 90 degrees
- moved R22 25.3 mm to (116.8, 103.9), turned to 90 degrees
- moved U6 21.4 mm to (121.0, 68.5)
- moved R14 18.3 mm to (131.6, 90.8)
- moved R10 17.8 mm to (119.0, 53.8)
- moved R17 17.3 mm to (100.0, 73.0), turned to 270 degrees
- moved R1 16.8 mm to (130.0, 121.2), turned to 270 degrees
- moved R8 16.1 mm to (105.0, 43.8)
- moved R15 14.7 mm to (101.8, 58.4), turned to 90 degrees
- moved R19 14.2 mm to (101.8, 105.3)
- moved R4 13.0 mm to (105.0, 47.0), turned to 0 degrees
- moved R6 10.8 mm to (119.0, 50.5), turned to 180 degrees
- moved R16 10.6 mm to (101.8, 64.0), turned to 270 degrees
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Connections:
- J2 pad 1: CV1_LED_OUT -> CV1_OUT
- J2 pad 2: CV1_OUT -> CV2_OUT
- J2 pad 3: CV2_LED_OUT -> CV3_OUT
- J2 pad 4: CV2_OUT -> CV4_OUT
- J2 pad 5: CV3_OUT -> CV1_LED_OUT
- J2 pad 6: CV3_LED_OUT -> CV2_LED_OUT
- J2 pad 7: CV4_OUT -> CV3_LED_OUT
- J4 pad 1: GND -> NRST
- J4 pad 3: GATE7_LED_OUT -> GND
- J4 pad 6: USB_VBUS -> USB_DP
- J4 pad 8: USB_DP -> USB_VBUS
- J5 pad 1: GND -> GATE7_LED_OUT
- J5 pad 6: NRST -> GND
- U1 pad 11: GATE6 -> Net-(U1-Pad11)
- U1 pad 15: GATE1 -> Net-(U1-Pad15)
- U1 pad 2: CV4_LED -> CV2_LED
- U1 pad 23: GATE4 -> GATE1
- U1 pad 25: GATE7 -> GATE4
- U1 pad 28: Net-(U1-Pad28) -> GATE6
- U1 pad 3: Net-(U1-Pad3) -> CV1_LED
- U1 pad 35: CV2_LED -> Net-(U1-Pad35)
- U1 pad 40: CV3_LED -> GATE7
- U1 pad 59: Net-(U1-Pad59) -> CV4_LED
- U1 pad 61: CV1_LED -> CV3_LED
- U3 pad 1: CV1_OUT -> CV3_OUT
- U3 pad 10: DAC_3 -> DAC_1
- U3 pad 2: Net-(R2-Pad2) -> Net-(R5-Pad2)
- U3 pad 3: DAC_1 -> DAC_3
- U3 pad 8: CV3_OUT -> CV1_OUT
- U3 pad 9: Net-(R5-Pad2) -> Net-(R2-Pad2)
- U6 pad 11: GATE5 -> GATE8
- U6 pad 12: GATE4_OUT -> GATE7_OUT
- U6 pad 14: GATE3_OUT -> GATE5_OUT
- U6 pad 15: GATE7 -> GATE4
- U6 pad 16: GATE2_OUT -> GATE3_OUT
- U6 pad 17: GATE8 -> GATE2
- U6 pad 3: GATE8_OUT -> GATE2_OUT
- U6 pad 4: GATE2 -> GATE3
- U6 pad 5: GATE7_OUT -> GATE4_OUT
- U6 pad 6: GATE3 -> GATE5
- U6 pad 8: GATE4 -> GATE7
- U6 pad 9: GATE5_OUT -> GATE8_OUT
- U7 pad 11: DAC_3 -> DAC_2
- U7 pad 14: DAC_2 -> DAC_3
- U7 pad 3: DAC_1 -> DAC_4
- U7 pad 6: DAC_4 -> DAC_1
Routing:
- net +3V3: track 50.4 -> 179.7 mm, vias 0 -> 6
- net VEE: track 6.31 -> 108.3 mm, vias 0 -> 2
- net GATE7_OUT: track 0.00 -> 75.1 mm, vias 0 -> 1
- net GATE5_OUT: track 0.00 -> 74.1 mm, vias 0 -> 1
- net +5V: track 5.43 -> 74.0 mm, vias 0 -> 3
- net GATE6_OUT: track 0.00 -> 68.1 mm, vias 0 -> 1
- net VCC: track 47.0 -> 113.5 mm, vias 0 -> 2
- net GATE8_OUT: track 0.00 -> 66.1 mm, vias 0 -> 1
- net GND: track 0.00 -> 56.1 mm, vias 0 -> 24
- net GATE1: track 3.02 -> 56.9 mm, vias 0 -> 3
- net NRST: track 3.33 -> 56.2 mm, vias 0 -> 2
- net GATE5: track 0.00 -> 48.8 mm, vias 0 -> 2
- net USB_VBUS: track 0.00 -> 48.5 mm
- net USB_DM: track 0.00 -> 45.6 mm
- net USB_DP: track 0.00 -> 42.8 mm
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
Commit message: Updated silkscreen
Parts:
- R1: value 220 -> 220R
- R11, R12, R13, R14, R16, R17, R19, R20, R21, R22: value 100 -> 100R
- R15: value 100 -> 100r
Other:
- board text added: "16"
- board text added: "3.3VA"
- board text added: "33"
- board text added: "49"
- board text added: "5V"
- board text added: "CV1 CV2 CV3 CV4"
- board text added: "G1L G1 G2L G2"
- board text added: "G3 G3L G4 G4L"
- board text added: "G5"
- board text added: "G5L"
- board text added: "G6"
- board text added: "G7"
- board text added: "G8"
- board text added: "GND"
- board text added: "MD"
- board text added: "MV"
- board text added: "RST"
- board text added: "UDM"
- board text added: "UDP"
- board text added: "UVB"

Commit message: Updated silkscreens and further PCB optimisations
Parts:
- J2: value Conn_01x08_Male -> Conn_01x09_Male; footprint Socket_Strips:Socket_Strip_Straight_1x08_Pitch2.54mm -> Socket_Strips:Socket_Strip_Straight_1x09_Pitch2.54mm
- R1: value 220R -> 220
- R11, R12, R13, R14, R16, R17, R19, R20, R21, R22: value 100R -> 100
- R15: value 100r -> 100
- moved J2 2.60 mm to (98.0, 47.4)
Connections:
- J2 pad 3: CV3_OUT -> GND
- J2 pad 4: CV4_OUT -> CV3_OUT
- J2 pad 5: CV1_LED_OUT -> CV4_OUT
- J2 pad 6: CV2_LED_OUT -> CV1_LED_OUT
- J2 pad 7: CV3_LED_OUT -> CV2_LED_OUT
- J2 pad 8: CV4_LED_OUT -> CV3_LED_OUT
Routing:
- net GND: track 56.1 -> 59.4 mm, vias 24 -> 28
- net +3V3: track 179.7 -> 182.9 mm
- net CV2_OUT: track 17.6 -> 15.2 mm
- net CV4_OUT: track 26.6 -> 28.7 mm
- net CV1_OUT: track 25.5 -> 26.9 mm
- net CV3_OUT: track 12.5 -> 11.9 mm
Other:
- board text added: "CV1-4 GND"
- board text added: "Mountjoy Modular MIDI Monger Electronics Board v1.0"
- board text removed: "CV1 CV2 CV3 CV4"

Commit message: First draft of PCBs completed and sent to JLC
Other:
- board text added: "CV LED1-4"
- board text added: "CV1"
- board text added: "CV2"
- board text added: "CV3"
- board text added: "CV4"
- board text removed: "CV1-4 GND"
Changed lines of the file:
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@@
   (general
     (thickness 1.6)
-    (drawings 34)
+    (drawings 40)
     (tracks 571)
     (zones 0)
@@
     (31 B.Cu signal)
     (32 B.Adhes user)
-    (33 F.Adhes user)
+    (33 F.Adhes user hide)
     (34 B.Paste user)
     (35 F.Paste user)
@@
   )
   (setup
-    (last_trace_width 0.3)
+    (last_trace_width 0.25)
     (user_trace_width 0.3)
     (user_trace_width 0.4)
@@
       (outputformat 1)
       (mirror false)
-      (drillshape 1)
+      (drillshape 0)
       (scaleselection 1)
-      (outputdirectory ""))
+      (outputdirectory "Electronics_PCB_Gerbers/"))
   )
   (net 0 "")
@@
     (descr "Through hole straight socket strip, 1x09, 2.54mm pitch, single row")
     (tags "Through hole socket strip THT 1x09 2.54mm single row")
-    (fp_text reference J2 (at 0 -2.33) (layer F.SilkS)
+    (fp_text reference J2 (at 0 -2.33) (layer F.SilkS) hide
       (effects (font (size 1 1) (thickness 0.15)))
     )
@@
     (tags "resistor 0805")
     (attr smd)
-    (fp_text reference R4 (at -3.5 0) (layer B.SilkS)
-      (effects (font (size 1 1) (thickness 0.15)) (justify mirror))
-    )
-    (fp_text value 10k (at 0 -1.75) (layer B.Fab)
+    (fp_text reference R4 (at 1.6 -1.4) (layer B.SilkS)
+      (effects (font (size 1 1) (thickness 0.15)) (justify mirror))
+    )
+    (fp_text value 10k (at -2.05 -1.4) (layer B.SilkS)
       (effects (font (size 1 1) (thickness 0.15)) (justify mirror))
     )
@@
     (tags "resistor 0805")
     (attr smd)
-    (fp_text reference R5 (at -3.5 -0.25) (layer B.SilkS)
-      (effects (font (size 1 1) (thickness 0.15)) (justify mirror))
-    )
-    (fp_text value 10k (at 0 -1.75) (layer B.Fab)
+    (fp_text reference R5 (at 1.7 -1.35) (layer B.SilkS)
+      (effects (font (size 1 1) (thickness 0.15)) (justify mirror))
+    )
+    (fp_text value 10k (at -2.1 -1.35) (layer B.SilkS)
       (effects (font (size 1 1) (thickness 0.15)) (justify mirror))
     )
@@
     (tags "resistor 0805")
     (attr smd)
-    (fp_text reference R8 (at -3.5 -0.25) (layer B.SilkS)
-      (effects (font (size 1 1) (thickness 0.15)) (justify mirror))
-    )
-    (fp_text value 2k (at 0 -1.75) (layer B.Fab)
+    (fp_text reference R8 (at 1.7 -1.35) (layer B.SilkS)
+      (effects (font (size 1 1) (thickness 0.15)) (justify mirror))
+    )
+    (fp_text value 2k (at -1.75 -1.35) (layer B.SilkS)
       (effects (font (size 1 1) (thickness 0.15)) (justify mirror))
     )
@@
     (tags "resistor 0805")
     (attr smd)
-    (fp_text reference R9 (at 3.5 0.25) (layer B.SilkS)
-      (effects (font (size 1 1) (thickness 0.15)) (justify mirror))
-    )
-    (fp_text value 2k (at 0 -1.75) (layer B.Fab)
+    (fp_text reference R9 (at -1.45 1.3) (layer B.SilkS)
+      (effects (font (size 1 1) (thickness 0.15)) (justify mirror))
+    )
+    (fp_text value 2k (at 1.7 1.3) (layer B.SilkS)
       (effects (font (size 1 1) (thickness 0.15)) (justify mirror))
     )
@@
     (tags "resistor 0805")
     (attr smd)
-    (fp_text reference R15 (at 0 1.7 90) (layer B.SilkS)
-      (effects (font (size 1 1) (thickness 0.15)) (justify mirror))
-    )
-    (fp_text value 100 (at 0 -1.75 90) (layer B.SilkS)
+    (fp_text reference R15 (at 1.5 1.6 90) (layer B.SilkS)
+      (effects (font (size 1 1) (thickness 0.15)) (justify mirror))
+    )
+    (fp_text value 100 (at -2 1.55 90) (layer B.SilkS)
       (effects (font (size 1 1) (thickness 0.15)) (justify mirror))
     )
@@
     )
   )
+  (gr_text CV4 (at 99.9 59.35 90) (layer B.SilkS)
+    (effects (font (size 1 1) (thickness 0.15)) (justify right mirror))
+  )
+  (gr_text CV3 (at 99.9 56 90) (layer B.SilkS)
+    (effects (font (size 1 1) (thickness 0.15)) (justify right mirror))
+  )
+  (gr_text CV2 (at 99.9 51.6 90) (layer B.SilkS)
+    (effects (font (size 1 1) (thickness 0.15)) (justify right mirror))
+  )
+  (gr_text CV1 (at 99.9 48.4 90) (layer B.SilkS)
+    (effects (font (size 1 1) (thickness 0.15)) (justify right mirror))
+  )
+  (gr_line (start 99.15 67.75) (end 99.15 60.15) (layer B.SilkS) (width 0.15))
+  (gr_line (start 100.7 67.75) (end 99.15 67.75) (layer B.SilkS) (width 0.15))
+  (gr_text "CV LED1-4" (at 100.85 67.75) (layer B.SilkS)
+    (effects (font (size 1 1) (thickness 0.15)) (justify right mirror))
+  )
   (gr_text "Mountjoy Modular\nMIDI Monger\nElectronics Board v1.0" (at 116.7 45.4) (layer F.SilkS)
     (effects (font (size 1.5 1.5) (thickness 0.3)))
@@
     (effects (font (size 1 1) (thickness 0.15)) (justify left mirror))
   )
-  (gr_text "CV1-4\nGND" (at 98.8 42.1) (layer B.SilkS)
-    (effects (font (size 1 1) (thickness 0.15)) (justify mirror))
-  )
   (gr_text MD (at 131.504762 135.425) (layer B.SilkS)
