File: Hardware/MidiMonger_panel.kicad_pcb (KiCad board)
At the start: 2 copper layers, 40.3 x 128.5 mm, 53 parts, among them J10 Gate8_Out, J11 CV1_Out, J12 CV2_Out, J13 CV3_Out, J14 CV4_Out, J15 USB_B_Wurth, J16 MIDI 5 Pin DIN, J2 Gate3_Out, J3 Gate4_Out, J4 Gate1_Out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

Commit message: First draft of PCBs completed and sent to JLC
Parts:
- removed D1: GATE1, LEDs:LED_D3.0mm
- removed D10: GATE6, LEDs:LED_D3.0mm
- removed D11: GATE7, LEDs:LED_D3.0mm
- removed D12: GATE8, LEDs:LED_D3.0mm
- removed D2: GATE2, LEDs:LED_D3.0mm
- removed D3: GATE3, LEDs:LED_D3.0mm
- removed D4: GATE4, LEDs:LED_D3.0mm
- removed D5: CV1, LEDs:LED_D3.0mm
- removed D6: CV2, LEDs:LED_D3.0mm
- removed D7: CV3, LEDs:LED_D3.0mm
- removed D8: CV4, LEDs:LED_D3.0mm
- removed D9: GATE5, LEDs:LED_D3.0mm
- removed J10: Gate8_Out, Custom_Footprints:Cliff_3.5mm_Stereo_Jack
- removed J11: CV1_Out, Custom_Footprints:Cliff_3.5mm_Stereo_Jack
- removed J12: CV2_Out, Custom_Footprints:Cliff_3.5mm_Stereo_Jack
- removed J13: CV3_Out, Custom_Footprints:Cliff_3.5mm_Stereo_Jack
- removed J14: CV4_Out, Custom_Footprints:Cliff_3.5mm_Stereo_Jack
- removed J15: USB_B_Wurth, Custom_Footprints:USB_B_Wurth
- removed J16: MIDI 5 Pin DIN, Custom_Footprints:MIDI_DIN
- removed J2: Gate3_Out, Custom_Footprints:Cliff_3.5mm_Stereo_Jack
- removed J3: Gate4_Out, Custom_Footprints:Cliff_3.5mm_Stereo_Jack
- removed J4: Gate1_Out, Custom_Footprints:Cliff_3.5mm_Stereo_Jack
- removed J5: Gate2_Out, Custom_Footprints:Cliff_3.5mm_Stereo_Jack
- removed J7: Gate5_Out, Custom_Footprints:Cliff_3.5mm_Stereo_Jack
- removed J8: Gate6_Out, Custom_Footprints:Cliff_3.5mm_Stereo_Jack
- removed J9: Gate7_Out, Custom_Footprints:Cliff_3.5mm_Stereo_Jack
- removed SW1: SW_Push, Buttons_Switches_THT:SW_PUSH_6mm
- added G***: LOGO, MIDI_Monger_logos:MIDIText, F.Cu at (107.3, 125.3)
- added G***: LOGO, MIDI_Monger_logos:MongerText, F.Cu at (125.1, 126.4)
- added Ref**: Oval_Mounting_Hole, Custom_Footprints:Oval_Mounting_Hole, F.Cu at (128.6, 33.8)
- added Ref**: Oval_Mounting_Hole, Custom_Footprints:Oval_Mounting_Hole, F.Cu at (103.4, 33.8)
- added Ref**: Oval_Mounting_Hole, Custom_Footprints:Oval_Mounting_Hole, F.Cu at (128.6, 156.3)
- added Ref**: Oval_Mounting_Hole, Custom_Footprints:Oval_Mounting_Hole, F.Cu at (103.4, 156.3)
- moved Ref** 2.02 mm to (116.0, 126.8)
- moved Ref** 2.00 mm to (101.0, 112.7)
- moved Ref** 2.00 mm to (101.0, 99.7)
- moved Ref** 2.00 mm to (123.5, 100.0)
- moved Ref** 2.00 mm to (123.5, 113.0)
- moved Ref** 2.00 mm to (108.5, 113.0)
- moved Ref** 2.00 mm to (108.5, 100.0)
- moved Ref** 2.00 mm to (131.0, 112.7)
- moved Ref** 2.00 mm to (131.0, 99.7)
- moved Ref** 1.00 mm to (125.0, 141.5)
Routing:
- net GATE7_LED_OUT: track 36.5 -> 0.00 mm
- net CV4_OUT: track 35.6 -> 0.00 mm
- net GATE6_OUT: track 29.7 -> 0.00 mm
- net GATE5_OUT: track 29.7 -> 0.00 mm
- net GND: track 29.6 -> 0.00 mm
- net GATE4_OUT: track 27.9 -> 0.00 mm
- net CV3_OUT: track 27.1 -> 0.00 mm
- net GATE5_LED_OUT: track 27.0 -> 0.00 mm
- net GATE6_LED_OUT: track 27.0 -> 0.00 mm
- net RESET_SWITCH: track 22.5 -> 0.00 mm
- net GATE3_OUT: track 20.0 -> 0.00 mm
- net CV1_LED_OUT: track 20.0 -> 0.00 mm
- net GATE8_OUT: track 19.2 -> 0.00 mm
- net GATE7_OUT: track 19.2 -> 0.00 mm
- net CV2_OUT: track 18.6 -> 0.00 mm
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- added copper zone on B.Cu, net (none)
- added copper zone on F.Cu, net (none)
- removed copper zone on B.Cu, net GND
- removed copper zone on F.Cu, net GND
Other:
- outline, holes or cut-outs redrawn
- board text added: "1"
- board text added: "2"
- board text added: "3"
- board text added: "4"
- board text added: "5"
- board text added: "6"
- board text added: "7"
- board text added: "8"
- board text added: "CV/Pitch"
- board text added: "Gate"
- board text added: "JLCJLCJLCJLC"
- board text added: "Mountjoy Modular"
- board text added: "Mountjoy Modular MIDI Monger Panel v1.0"
