File: Hardware/QMidiMonger_controls.kicad_pcb (KiCad board)
At the start: 2 copper layers, 40 x 102.5 mm, 26 parts, among them J1 CV_Out, J2 CV_Out, J20 Conn_01x09_Female, J21 Conn_01x08_Female, J22 Conn_01x08_Female, J23 Conn_01x03_Female, J3 CV_Out, J4 Gate_Out, J5 Gate_Out, J6 Gate_Out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

Commit message: Normalised audio to all CV returns
Connections:
- J1 pad 5: unconnected-(J1-Pad5) -> /AUDIO_IN1
- J1 pad 6: unconnected-(J1-Pad6) -> /AUDIO_IN2
- J1 pad 7: unconnected-(J1-Pad7) -> /AUDIO_IN3
- J1 pad 8: unconnected-(J1-Pad8) -> /AUDIO_IN4
- J2 pad 5: unconnected-(J2-Pad5) -> /AUDIO_IN1
- J2 pad 6: unconnected-(J2-Pad6) -> /AUDIO_IN2
- J2 pad 7: unconnected-(J2-Pad7) -> /AUDIO_IN3
- J2 pad 8: unconnected-(J2-Pad8) -> /AUDIO_IN4
Routing:
- net /AUDIO_IN4: track 27.5 -> 72.1 mm
- net /AUDIO_IN3: track 29.5 -> 67.6 mm
- net /AUDIO_IN1: track 37.1 -> 75.2 mm
- net /AUDIO_IN2: track 34.6 -> 72.7 mm
